Commit message: Sync everything to the remote, roughly organized
This is not a finished cleanup pass.  I'm pushing so I have all of it on
my local machine: the new sibling trees (dataset_builders/, analysis/,
docs/), the runtime modules, and the objhead training code.  Everything
here is roughly organized and I'll review it all personally later.

File: giava.urdf (robot description, URDF)
Before this commit: robot giava, 31 links, 30 joints
Links:
- added link left_gripper_camera, mass 0.421580; collision mesh filename=aloha_assets/d405_solid.stl; visual mesh filename=aloha_assets/d405_solid.stl
- added link left_gripper_plate, mass 0.421580; collision mesh filename=aloha_assets/vx300s_7_gripper_bar.stl; collision mesh filename=aloha_assets/vx300s_7_gripper_prop.stl
- added link right_gripper_camera, mass 0.421580; collision mesh filename=aloha_assets/d405_solid.stl; visual mesh filename=aloha_assets/d405_solid.stl
- added link right_gripper_plate, mass 0.421580; collision mesh filename=aloha_assets/vx300s_7_gripper_bar.stl; collision mesh filename=aloha_assets/vx300s_7_gripper_prop.stl
- link left_gripper_base: geometry collision mesh filename=aloha_assets/vx300s_7_gripper_wrist_mount.stl; visual mesh filename=aloha_assets/vx300s_7_gripper_wrist_mount.stl
- link left_left_finger_link: geometry collision box size=0.0103 0.0100 0.0164; collision mesh filename=aloha_assets/vx300s_8_custom_finger_right.stl
- link left_right_finger_link: geometry collision box size=0.0102 0.0101 0.0164; collision mesh filename=aloha_assets/vx300s_8_custom_finger_left.stl
- link right_gripper_base: geometry collision mesh filename=aloha_assets/vx300s_7_gripper_wrist_mount.stl; visual mesh filename=aloha_assets/vx300s_7_gripper_wrist_mount.stl
- link right_left_finger_link: geometry collision box size=0.0103 0.0100 0.0164; collision mesh filename=aloha_assets/vx300s_8_custom_finger_right.stl
- link right_right_finger_link: geometry collision box size=0.0102 0.0101 0.0164; collision mesh filename=aloha_assets/vx300s_8_custom_finger_left.stl
Joints:
- added joint left_gripper_camera_fixed: type fixed, parent left_gripper_base, child left_gripper_camera, origin xyz=0.0 0.0 0.0 rpy=0.0 0.0 0.0
- added joint left_gripper_plate_fixed: type fixed, parent left_gripper_base, child left_gripper_plate, origin xyz=0.0 0.0 0.0 rpy=0.0 0.0 0.0
- added joint right_gripper_camera_fixed: type fixed, parent right_gripper_base, child right_gripper_camera, origin xyz=0.0 0.0 0.0 rpy=0.0 0.0 0.0
- added joint right_gripper_plate_fixed: type fixed, parent right_gripper_base, child right_gripper_plate, origin xyz=0.0 0.0 0.0 rpy=0.0 0.0 0.0
- joint base_left_base_link_fixed: origin xyz=0.520000 -0.019000 0.020000 rpy=0.000000 0.000000 3.141593 -> xyz=0.535278 -0.020820 0.045371 rpy=0.000000 0.000000 3.137374
- joint left_left_finger: origin xyz=0.019100 -0.014164 0.021173 rpy=-1.570796 0.000000 1.570796 -> xyz=0.019100 0.014164 0.021173 rpy=1.570796 0.000000 -1.570797
- joint left_right_finger: origin xyz=-0.019100 -0.014164 0.021173 rpy=1.570796 0.000000 1.570796 -> xyz=-0.019100 0.014164 0.021173 rpy=-1.570796 0.000000 -1.570797
- joint middle_lower_forearm: axis 2.8698592549372254e-42 -1.0 7.97360475549766e-14 -> 0.0 -1.0 0.0; limit lower=-1.7453292519943295 upper=2.1467549799530254 effort=5 velocity=3.141592653589793 -> lower=-1.6553292519943295 upper=2.2367549799530253 effort=5 velocity=3.141592653589793; origin xyz=0.0782 0.0 0.019100000000000002 rpy=1.5707963267949763 -0.0 1.5707963267948966 -> xyz=0.0782 0.0 0.019100000000000002 rpy=1.570796326794976 0.0 1.6607963267948964
- joint middle_pan: axis 0.0 -6.162975822039155e-33 1.0 -> 0.0 0.0 1.0; limit lower=-3.141592653589793 upper=0.915 effort=1 velocity=3.141592653589793 -> lower=-0.7565926535897933 upper=3.3 effort=1 velocity=3.141592653589793; origin xyz=0.04125 0.03725000000000001 1.1379786002407855e-17 rpy=-1.5707963267948963 2.5199808612277694e-29 -1.4272358353620772e-42 -> xyz=0.04125 0.03725000000000001 1.1379786002407855e-17 rpy=1.5707963267948966 -0.7565926535897937 -3.141592653589793
- joint middle_shoulder: axis 0.0 -1.0 0.0 -> 0.0 1.0 0.0; limit lower=-1.8849555921538759 upper=1.9896753472735358 effort=20 velocity=3.141592653589793 -> lower=-2.3046753472735357 upper=1.569955592153876 effort=20 velocity=3.141592653589793; origin xyz=0.0 0.013999999999999999 0.04125 rpy=-0.0 -1.5707963267948966 0 -> xyz=0.0 0.013999999999999999 0.04125 rpy=0.0 -1.4757963267948964 0.0
- joint middle_upper_arm: axis -2.8698592549372254e-42 -1.0 -2.1791458186645675e-52 -> 0.0 1.0 0.0; limit lower=-2.1467549799530254 upper=1.6057029118347832 effort=15 velocity=3.141592653589793 -> lower=-1.735702911834783 upper=2.0167549799530256 effort=15 velocity=3.141592653589793; origin xyz=0.25 0.0 -0.05 rpy=2.1791458186645653e-52 -1.4349296274686127e-42 2.8698592549372254e-42 -> xyz=0.25 0.0 -0.05 rpy=0.0 -0.04999999999999988 0.0
- joint middle_upper_forearm: axis 1.0 -1.4349296274686127e-42 2.1791458186645653e-52 -> 1.0 0.0 0.0; limit lower=-3.141582653589793 upper=3.141582653589793 effort=2 velocity=3.141592653589793 -> lower=-3.211582653589793 upper=3.071582653589793 effort=2 velocity=3.141592653589793; origin xyz=0.0 -0.013499999999999998 -0.1718 rpy=1.5707963267948966 1.5707963267948966 0 -> xyz=0.0 -0.013499999999999998 -0.1718 rpy=1.6407963267948966 1.5707963267948966 0.0
- joint middle_wrist: axis 1.0 -1.4349446804892014e-42 1.6339707364920764e-13 -> 1.0 0.0 0.0; limit lower=-3.141592653589793 upper=3.141592653589793 effort=1 velocity=3.141592653589793 -> lower=-1.581592653589793 upper=4.701592653589794 effort=1 velocity=3.141592653589793; origin xyz=-1.7053025658242404e-15 -0.01899999999999482 0.06500000000000149 rpy=-1.570796326794897 -1.5707963267948128 0 -> xyz=-1.7053025658242404e-15 -0.01899999999999482 0.06500000000000149 rpy=-3.130796326794897 -1.5707963267948128 0.0
- joint right_left_finger: origin xyz=0.019100 -0.014164 0.021173 rpy=-1.570796 0.000000 1.570796 -> xyz=0.019100 0.014164 0.021173 rpy=1.570796 0.000000 -1.570797
- joint right_right_finger: origin xyz=-0.019100 -0.014164 0.021173 rpy=1.570796 0.000000 1.570796 -> xyz=-0.019100 0.014164 0.021173 rpy=-1.570796 0.000000 -1.570797

File: interbotix_ws/src/interbotix_ros_manipulators/interbotix_ros_xsarms/interbotix_xsarm_descriptions/urdf/vx300s.urdf.xacro (robot description, xacro)
@@ -38,9 +38,22 @@
       </geometry>
     </collision>
-    <inertial>
-      <origin rpy="0 0 ${pi/2}" xyz="-0.0534774000 -0.0005625750 0.0205961000"/>
-      <mass value="0.969034" />
-      <inertia ixx="0.0060240000" iyy="0.0017000000" izz="0.0071620000" ixy="0.0000471300" ixz="0.0000038510" iyz="-0.0000841500" />
-    </inertial>
+    <!-- NO inertial block on this link, DELIBERATELY (2026-08-27).
+         This is the ROOT link of the description, and KDL does not support a
+         root link with an inertia: robot_state_publisher warned about it on
+         every launch, once per arm.
+         ("The root link ... has an inertia specified in the URDF, but KDL
+          does not support a root link with an inertia. As a workaround, you
+          can add an extra dummy link to your URDF.")
+         Nothing in this stack reads link inertia. pyroki is kinematics only,
+         the xs_sdk commands servo positions, and the collision models are
+         built from the meshes, so removing it changes no behaviour and
+         removes the warning at its source.
+         The upstream workaround, use_world_frame:=true, adds a massless
+         `world` parent instead. NOT used here: three arms each publishing
+         `world` at identity relative to their own base would put one TF frame
+         in three different physical places.
+         It would only matter under load_gazebo_configs, which this rig never
+         launches, and a fixed-base root is static there anyway. If you ever do
+         simulate, restore the inertial here or add the dummy link. -->
   </link>
   <joint name="waist" type="revolute">
@@ -83,5 +96,8 @@
   <joint name="shoulder" type="revolute">
     <axis xyz="0 1 0"/>
-    <limit effort="20" lower="${radians(-106)}" upper="${radians(72)}" velocity="${pi}"/>
+    <!-- lower widened -106 -> -112 deg (2026-08): the deployed reset poses
+         command shoulder -1.90 rad, 0.05 past the stock limit.  Matching
+         widening in xsarm_control/config/vx300s.yaml (servo registers). -->
+    <limit effort="20" lower="${radians(-112)}" upper="${radians(72)}" velocity="${pi}"/>
     <origin rpy="0 0 0" xyz="0 0 0.04805"/>
     <parent link="$(arg robot_name)/shoulder_link"/>
@@ -120,5 +136,8 @@
   <joint name="elbow" type="revolute">
     <axis xyz="0 1 0"/>
-    <limit effort="15" lower="${radians(-101)}" upper="${radians(92)}" velocity="${pi}"/>
+    <!-- upper widened 92 -> 98 deg (2026-08): deployed poses command elbow
+         1.63 rad, 0.03 past stock.  Matching servo registers in
+         xsarm_control/config/vx300s.yaml. -->
+    <limit effort="15" lower="${radians(-101)}" upper="${radians(98)}" velocity="${pi}"/>
     <origin rpy="0 0 0" xyz="0.05955 0 0.3"/>
     <parent link="$(arg robot_name)/upper_arm_link"/>

File: interbotix_ws/src/wx250s_7dof_description/urdf/wx250s_7dof.urdf (robot description, URDF)
Before this commit: robot wx250s_6dof, 8 links, 7 joints
Joints:
- joint camera_yaw: limit lower=-3.10 upper=3.07 effort=1 velocity=3.141592653589793 -> lower=-3.10 upper=3.30 effort=1 velocity=3.141592653589793
- joint waist: limit lower=-6.35 upper=0.00 effort=10 velocity=3.141592653589793 -> lower=-4.90 upper=4.90 effort=10 velocity=3.141592653589793

File: interbotix_ws/src/wx250s_7dof_description/urdf/wx250s_7dof.urdf.xacro (robot description, xacro)
@@ -28,23 +28,45 @@
       <origin rpy="0 0 ${pi/2}" xyz="0 0 0"/>
       <geometry>
-        <mesh filename="package://wx250s_7dof_description/meshes/430-Base-v3.stl" scale="0.001 0.001 0.001"/>
-      </geometry>
-      <material name="interbotix_black"/>
-    </visual>
-    <collision>
-      <origin rpy="0 0 ${pi/2}" xyz="0 0 0"/>
-      <geometry>
-        <mesh filename="package://wx250s_7dof_description/meshes/430-Base-v3.stl" scale="0.001 0.001 0.001"/>
-      </geometry>
-    </collision>
-    <inertial>
-      <origin rpy="0 0 ${pi/2}" xyz="-0.0380446000 0.0006138920 0.0193354000"/>
-      <mass value="0.538736" />
-      <inertia ixx="0.0021150000" iyy="0.0006921000" izz="0.0025240000" ixy="-0.0000163500" ixz="0.0000006998" iyz="0.0000464200" />
-    </inertial>
+        <mesh filename="package://wx250s_7dof_description/urdf/meshes/430-Base-v3.stl" scale="0.001 0.001 0.001"/>
+      </geometry>
+      <material name="interbotix_black"/>
+    </visual>
+    <collision>
+      <origin rpy="0 0 ${pi/2}" xyz="0 0 0"/>
+      <geometry>
+        <mesh filename="package://wx250s_7dof_description/urdf/meshes/430-Base-v3.stl" scale="0.001 0.001 0.001"/>
+      </geometry>
+    </collision>
+    <!-- NO inertial block on this link, DELIBERATELY (2026-08-27).
+         This is the ROOT link of the description, and KDL does not support a
+         root link with an inertia: robot_state_publisher warned about it on
+         every launch, once per arm.
+         ("The root link ... has an inertia specified in the URDF, but KDL
+          does not support a root link with an inertia. As a workaround, you
+          can add an extra dummy link to your URDF.")
+         Nothing in this stack reads link inertia. pyroki is kinematics only,
+         the xs_sdk commands servo positions, and the collision models are
+         built from the meshes, so removing it changes no behaviour and
+         removes the warning at its source.
+         The upstream workaround, use_world_frame:=true, adds a massless
+         `world` parent instead. NOT used here: three arms each publishing
+         `world` at identity relative to their own base would put one TF frame
+         in three different physical places.
+         It would only matter under load_gazebo_configs, which this rig never
+         launches, and a fixed-base root is static there anyway. If you ever do
+         simulate, restore the inertial here or add the dummy link. -->
   </link>
   <joint name="waist" type="revolute">
     <axis xyz="0 0 1"/>
-    <limit effort="10" lower="-6.35" upper="0.00" velocity="${pi}"/>
+    <!-- The rest pose sits ON the encoder's single-turn seam (assembly), so
+             the boot reading flips between +3.14 and -3.14 depending on which
+             side the gearbox settles it is NOT a one-time frame change.
+             The [-6.35, 0] -> [0, 6.35] remap (2026-08) patched one boot side
+             and broke the other.  These limits admit BOTH labels plus ~1.75
+             rad of yaw around camera-forward; the waist runs in ext_position
+             mode (puppet_modes_middle.yaml) so commands may cross the seam,
+             and software always targets the 2pi-equivalent nearest the
+             current reading, so no long sweeps are commandable. -->
+        <limit effort="10" lower="-4.90" upper="4.90" velocity="${pi}"/>
     <origin rpy="0 0 0" xyz="0 0 0.072"/>
     <parent link="$(arg robot_name)/$(arg base_link_frame)"/>
@@ -65,5 +87,5 @@
       <origin rpy="0 0 ${pi/2}" xyz="0 0 -0.003"/>
       <geometry>
-        <mesh filename="package://wx250s_7dof_description/meshes/430-Dual-Shoulder-v2.stl" scale="0.001 0.001 0.001"/>
+        <mesh filename="package://wx250s_7dof_description/urdf/meshes/430-Dual-Shoulder-v2.stl" scale="0.001 0.001 0.001"/>
       </geometry>
       <material name="interbotix_black"/>
@@ -72,5 +94,5 @@
       <origin rpy="0 0 ${pi/2}" xyz="0 0 -0.003"/>
       <geometry>
-        <mesh filename="package://wx250s_7dof_description/meshes/430-Dual-Shoulder-v2.stl" scale="0.001 0.001 0.001"/>
+        <mesh filename="package://wx250s_7dof_description/urdf/meshes/430-Dual-Shoulder-v2.stl" scale="0.001 0.001 0.001"/>
       </geometry>
     </collision>
@@ -102,12 +124,12 @@
       <origin rpy="0 0 ${pi/2}" xyz="0 0 0"/>
       <geometry>
-        <mesh filename="package://wx250s_7dof_description/meshes/UA---6---WX-250-v2.stl" scale="0.001 0.001 0.001"/>
-      </geometry>
-      <material name="interbotix_black"/>
-    </visual>
-    <collision>
-      <origin rpy="0 0 ${pi/2}" xyz="0 0 0"/>
-      <geometry>
-        <mesh filename="package://wx250s_7dof_description/meshes/UA---6---WX-250-v2.stl" scale="0.001 0.001 0.001"/>
+        <mesh filename="package://wx250s_7dof_description/urdf/meshes/UA---6---WX-250-v2.stl" scale="0.001 0.001 0.001"/>
+      </geometry>
+      <material name="interbotix_black"/>
+    </visual>
+    <collision>
+      <origin rpy="0 0 ${pi/2}" xyz="0 0 0"/>
+      <geometry>
+        <mesh filename="package://wx250s_7dof_description/urdf/meshes/UA---6---WX-250-v2.stl" scale="0.001 0.001 0.001"/>
       </geometry>
     </collision>
@@ -139,5 +161,5 @@
       <origin rpy="0 0 0" xyz="0 0 0"/>
       <geometry>
-        <mesh filename="package://wx250s_7dof_description/meshes/SIMPLIFIED---WXA-250-6DOF-Upper-Forearm-v3.stl" scale="0.001 0.001 0.001"/>
+        <mesh filename="package://wx250s_7dof_description/urdf/meshes/SIMPLIFIED---WXA-250-6DOF-Upper-Forearm-v3.stl" scale="0.001 0.001 0.001"/>
       </geometry>
       <material name="interbotix_black"/>
@@ -146,5 +168,5 @@
       <origin rpy="0 0 0" xyz="0 0 0"/>
       <geometry>
-        <mesh filename="package://wx250s_7dof_description/meshes/SIMPLIFIED---WXA-250-6DOF-Upper-Forearm-v3.stl" scale="0.001 0.001 0.001"/>
+        <mesh filename="package://wx250s_7dof_description/urdf/meshes/SIMPLIFIED---WXA-250-6DOF-Upper-Forearm-v3.stl" scale="0.001 0.001 0.001"/>
       </geometry>
     </collision>
@@ -176,5 +198,5 @@
       <origin rpy="${pi} 0 0" xyz="0 0 0"/>
       <geometry>
-        <mesh filename="package://wx250s_7dof_description/meshes/SIMPLIFIED---WXA-250-6DOF-Lower-Forearm-v4.stl" scale="0.001 0.001 0.001"/>
+        <mesh filename="package://wx250s_7dof_description/urdf/meshes/SIMPLIFIED---WXA-250-6DOF-Lower-Forearm-v4.stl" scale="0.001 0.001 0.001"/>
       </geometry>
       <material name="interbotix_black"/>
@@ -183,5 +205,5 @@
       <origin rpy="${pi} 0 0" xyz="0 0 0"/>
       <geometry>
-        <mesh filename="package://wx250s_7dof_description/meshes/SIMPLIFIED---WXA-250-6DOF-Lower-Forearm-v4.stl" scale="0.001 0.001 0.001"/>
+        <mesh filename="package://wx250s_7dof_description/urdf/meshes/SIMPLIFIED---WXA-250-6DOF-Lower-Forearm-v4.stl" scale="0.001 0.001 0.001"/>
       </geometry>
     </collision>
@@ -213,12 +235,12 @@
       <origin rpy="0 0 ${pi/2}" xyz="0 0 0"/>
       <geometry>
-        <mesh filename="package://wx250s_7dof_description/meshes/430---Wrist-v3.stl" scale="0.001 0.001 0.001"/>
-      </geometry>
-      <material name="interbotix_black"/>
-    </visual>
-    <collision>
-      <origin rpy="0 0 ${pi/2}" xyz="0 0 0"/>
-      <geometry>
-        <mesh filename="package://wx250s_7dof_description/meshes/430---Wrist-v3.stl" scale="0.001 0.001 0.001"/>
+        <mesh filename="package://wx250s_7dof_description/urdf/meshes/430---Wrist-v3.stl" scale="0.001 0.001 0.001"/>
+      </geometry>
+      <material name="interbotix_black"/>
+    </visual>
+    <collision>
+      <origin rpy="0 0 ${pi/2}" xyz="0 0 0"/>
+      <geometry>
+        <mesh filename="package://wx250s_7dof_description/urdf/meshes/430---Wrist-v3.stl" scale="0.001 0.001 0.001"/>
       </geometry>
     </collision>
@@ -249,10 +271,10 @@
       <origin xyz="0 0 0" rpy="0 0 0"/>
       <geometry>
-        <mesh filename="package://wx250s_7dof_description/meshes/430---Wrist-v3.stl" scale="0.001 0.001 0.001"/>
-      </geometry>
-    </visual>
-    <collision>
-      <geometry>
-        <mesh filename="package://wx250s_7dof_description/meshes/430---Wrist-v3.stl" scale="0.001 0.001 0.001"/>
+        <mesh filename="package://wx250s_7dof_description/urdf/meshes/430---Wrist-v3.stl" scale="0.001 0.001 0.001"/>
+      </geometry>
+    </visual>
+    <collision>
+      <geometry>
+        <mesh filename="package://wx250s_7dof_description/urdf/meshes/430---Wrist-v3.stl" scale="0.001 0.001 0.001"/>
       </geometry>
     </collision>
@@ -265,5 +287,5 @@
   <joint name="camera_yaw" type="revolute">
     <axis xyz="0 0 1"/>
-    <limit effort="1" lower="-3.10" upper="3.07" velocity="${pi}"/>
+    <limit effort="1" lower="-3.10" upper="3.30" velocity="${pi}"/>
     <origin xyz="0 0 0" rpy="0 0 0"/>
     <parent link="$(arg robot_name)/camera_roll_link"/>
@@ -282,10 +304,10 @@
     <visual>
       <geometry>
-        <mesh filename="package://wx250s_7dof_description/meshes/middlecamera.stl" scale="0.001 0.001 0.001"/>
-      </geometry>
-    </visual>
-    <collision>
-      <geometry>
-        <mesh filename="package://wx250s_7dof_description/meshes/middlecamera.stl" scale="0.001 0.001 0.001"/>
+        <mesh filename="package://wx250s_7dof_description/urdf/meshes/middlecamera.stl" scale="0.001 0.001 0.001"/>
+      </geometry>
+    </visual>
+    <collision>
+      <geometry>
+        <mesh filename="package://wx250s_7dof_description/urdf/meshes/middlecamera.stl" scale="0.001 0.001 0.001"/>
       </geometry>
     </collision>
